File: Buttons.kicad_sch (KiCad schematic)
At the start: 20 parts, among them J1001 buttons, J1002 buttons, J1003 buttons, J1004 buttons, J1005 buttons, SW1001 switch, SW1002 switch, SW1003 switch, SW1004 switch, SW1005 switch

Commit message: feat: migrar a KiCad 10 y reemplazar 0603 por 0805 - actualizar versiones de archivos y footprints SMD
Parts:
- R? (x10): footprint Resistor_SMD:R_0603_1608Metric -> Resistor_SMD:R_0805_2012Metric
