File: Display_Oled.kicad_sch (KiCad schematic)
At the start: 4 parts, among them J301 OledSpiST1306, J302 OledSpiST7789

Commit message: feat: migrar a KiCad 10 y reemplazar 0603 por 0805 - actualizar versiones de archivos y footprints SMD
Parts:
- R? (x2): footprint Resistor_SMD:R_0603_1608Metric -> Resistor_SMD:R_0805_2012Metric
