File: Display_Oled.kicad_sch (KiCad schematic)
At the start: 4 parts, among them J301 OledSpiST1306, J302 OledSpiST7789

Commit message: feat: agregar hierarchical_labels con nombres correctos a oS_AnaloDev (DiscoveryAnalog3) - 30 pines
Parts:
- gave numbers to parts that had none: 2
Changed lines of the file:
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@@
 		(in_pos_files yes)
 		(dnp no)
-		(property "Reference" "R?"
+		(property "Reference" "R301"
 			(at 143.2052 91.7448 90)
 			(show_name no)
@@
 		(instances
 			(project "amper_volt_meter"
-				(path "/606ef755-236d-4283-a129-fc8150c20746/283e249b-17fa-4123-ad59-a4970e9d33a5"
-					(reference "#PWR?")
-					(unit 1)
-				)
 				(path "/606ef755-236d-4283-a129-fc8150c20746/f62fc848-fb80-4104-826c-eb02129eaaef"
 					(reference "#PWR0306")
@@
 		(in_pos_files yes)
 		(dnp no)
-		(property "Reference" "R?"
+		(property "Reference" "R302"
 			(at 152.0952 91.7448 90)
 			(show_name no)
