File: Display_Oled_Left.kicad_sch (KiCad schematic)
At the start: 5 parts, among them J701 OledSpiST7789, J702 OledSpiST1306

Commit message: feat: agregar hierarchical_labels con nombres correctos a oS_AnaloDev (DiscoveryAnalog3) - 30 pines
Parts:
- gave numbers to parts that had none: 2
Changed lines of the file:
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@@
 		(dnp no)
 		(fields_autoplaced yes)
-		(property "Reference" "#PWR?"
+		(property "Reference" "#PWR0704"
 			(at 138.303 77.216 0)
 			(hide yes)
@@
 				(path "/606ef755-236d-4283-a129-fc8150c20746/283e249b-17fa-4123-ad59-a4970e9d33a5"
 					(reference "#PWR0704")
-					(unit 1)
-				)
-				(path "/606ef755-236d-4283-a129-fc8150c20746/f62fc848-fb80-4104-826c-eb02129eaaef"
-					(reference "#PWR?")
 					(unit 1)
 				)
@@
 		(dnp no)
 		(fields_autoplaced yes)
-		(property "Reference" "#PWR?"
+		(property "Reference" "#PWR0702"
 			(at 96.012 76.962 0)
 			(hide yes)
@@
 				(path "/606ef755-236d-4283-a129-fc8150c20746/283e249b-17fa-4123-ad59-a4970e9d33a5"
 					(reference "#PWR0702")
-					(unit 1)
-				)
-				(path "/606ef755-236d-4283-a129-fc8150c20746/f62fc848-fb80-4104-826c-eb02129eaaef"
-					(reference "#PWR?")
 					(unit 1)
 				)
@@
 		(dnp no)
 		(fields_autoplaced yes)
-		(property "Reference" "#PWR?"
+		(property "Reference" "#PWR0703"
 			(at 114.3 77.216 0)
 			(hide yes)
@@
 				(path "/606ef755-236d-4283-a129-fc8150c20746/283e249b-17fa-4123-ad59-a4970e9d33a5"
 					(reference "#PWR0703")
-					(unit 1)
-				)
-				(path "/606ef755-236d-4283-a129-fc8150c20746/f62fc848-fb80-4104-826c-eb02129eaaef"
-					(reference "#PWR?")
 					(unit 1)
 				)
@@
 		(in_pos_files yes)
 		(dnp no)
-		(property "Reference" "R?"
+		(property "Reference" "R702"
 			(at 131.953 87.376 90)
 			(show_name no)
@@
 				(path "/606ef755-236d-4283-a129-fc8150c20746/283e249b-17fa-4123-ad59-a4970e9d33a5"
 					(reference "R702")
-					(unit 1)
-				)
-				(path "/606ef755-236d-4283-a129-fc8150c20746/f62fc848-fb80-4104-826c-eb02129eaaef"
-					(reference "R?")
 					(unit 1)
 				)
@@
 		(dnp no)
 		(fields_autoplaced yes)
-		(property "Reference" "#PWR?"
+		(property "Reference" "#PWR0706"
 			(at 154.813 89.916 0)
 			(hide yes)
@@
 				(path "/606ef755-236d-4283-a129-fc8150c20746/283e249b-17fa-4123-ad59-a4970e9d33a5"
 					(reference "#PWR0706")
-					(unit 1)
-				)
-				(path "/606ef755-236d-4283-a129-fc8150c20746/f62fc848-fb80-4104-826c-eb02129eaaef"
-					(reference "#PWR?")
 					(unit 1)
 				)
@@
 		(dnp no)
 		(fields_autoplaced yes)
-		(property "Reference" "J?"
+		(property "Reference" "J702"
 			(at 168.783 102.616 0)
 			(show_name no)
@@
 				(path "/606ef755-236d-4283-a129-fc8150c20746/283e249b-17fa-4123-ad59-a4970e9d33a5"
 					(reference "J702")
-					(unit 1)
-				)
-				(path "/606ef755-236d-4283-a129-fc8150c20746/f62fc848-fb80-4104-826c-eb02129eaaef"
-					(reference "J?")
 					(unit 1)
 				)
@@
 		(dnp no)
 		(fields_autoplaced yes)
-		(property "Reference" "#PWR?"
+		(property "Reference" "#PWR0707"
 			(at 154.813 122.936 0)
 			(hide yes)
@@
 				(path "/606ef755-236d-4283-a129-fc8150c20746/283e249b-17fa-4123-ad59-a4970e9d33a5"
 					(reference "#PWR0707")
-					(unit 1)
-				)
-				(path "/606ef755-236d-4283-a129-fc8150c20746/f62fc848-fb80-4104-826c-eb02129eaaef"
-					(reference "#PWR?")
 					(unit 1)
 				)
@@
 		(in_pos_files yes)
 		(dnp no)
-		(property "Reference" "R?"
+		(property "Reference" "R701"
 			(at 123.063 87.376 90)
 			(show_name no)
@@
 				(path "/606ef755-236d-4283-a129-fc8150c20746/283e249b-17fa-4123-ad59-a4970e9d33a5"
 					(reference "R701")
-					(unit 1)
-				)
-				(path "/606ef755-236d-4283-a129-fc8150c20746/f62fc848-fb80-4104-826c-eb02129eaaef"
-					(reference "R?")
 					(unit 1)
 				)
@@
 		(dnp no)
 		(fields_autoplaced yes)
-		(property "Reference" "#PWR?"
+		(property "Reference" "#PWR0705"
 			(at 143.383 98.806 0)
 			(hide yes)
@@
 					(unit 1)
 				)
-				(path "/606ef755-236d-4283-a129-fc8150c20746/f62fc848-fb80-4104-826c-eb02129eaaef"
-					(reference "#PWR?")
-					(unit 1)
-				)
