File: Leds_Ports.kicad_sch (KiCad schematic)
At the start: 8 parts

Commit message: feat: migrar a KiCad 10 y reemplazar 0603 por 0805 - actualizar versiones de archivos y footprints SMD
Parts:
- R? (x4): footprint Resistor_SMD:R_0603_1608Metric -> Resistor_SMD:R_0805_2012Metric
