File: Leds_Ports.kicad_sch (KiCad schematic)
At the start: 8 parts

Commit message: feat: agregar hierarchical_labels con nombres correctos a oS_AnaloDev (DiscoveryAnalog3) - 30 pines
Parts:
- gave numbers to parts that had none: 4
Changed lines of the file:
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@@
 		(in_pos_files yes)
 		(dnp no)
-		(property "Reference" "R?"
+		(property "Reference" "R901"
 			(at 112.395 104.013 90)
 			(show_name no)
@@
 		(in_pos_files yes)
 		(dnp no)
-		(property "Reference" "R?"
+		(property "Reference" "R902"
 			(at 127.635 104.013 90)
 			(show_name no)
@@
 		(in_pos_files yes)
 		(dnp no)
-		(property "Reference" "R?"
+		(property "Reference" "R904"
 			(at 155.575 104.013 90)
 			(show_name no)
@@
 		(in_pos_files yes)
 		(dnp no)
-		(property "Reference" "R?"
+		(property "Reference" "R903"
 			(at 141.605 104.013 90)
 			(show_name no)
