File: PIM100.kicad_sch (KiCad schematic)
At the start: 10 parts, among them U1101 .

Commit message: feat: migrar a KiCad 10 y reemplazar 0603 por 0805 - actualizar versiones de archivos y footprints SMD
Parts:
- C1101, C1102, C1103, C1104, C1105, C1106, C1107, C1108, C1109: footprint Capacitor_SMD:C_0603_1608Metric -> Capacitor_SMD:C_0805_2012Metric
