File: PIM100.kicad_sch (KiCad schematic)
At the start: 10 parts, among them U1101 .

Commit message: feat: PIM100 - labels en mayusculas y pines externos ordenados por puerto (85 pines, 42 izq + 43 der)
Connections:
- net mclr renamed MCLR
- net osc1 renamed OSC1
- net osc2 renamed OSC2
- net ra10 renamed RA10
- net ra14 renamed RA14
- net ra15 renamed RA15
- net ra6 renamed RA6
- net ra7 renamed RA7
- net ra9 renamed RA9
- net rb10 renamed RB10
- net rb11 renamed RB11
- net rb12 renamed RB12
- net rb13 renamed RB13
- net rb14 renamed RB14
- net rb15 renamed RB15
- net rb8 renamed RB8
- net rb9 renamed RB9
- net rc13 renamed RC13
- net rc14 renamed RC14
- net rd10 renamed RD10
- net rd11 renamed RD11
- net rd12 renamed RD12
- net rd13 renamed RD13
- net rd14 renamed RD14
- net rd15 renamed RD15
- net rd8 renamed RD8
- net rd9 renamed RD9
- net re6 renamed RE6
- net re7 renamed RE7
- net re8 renamed RE8
- net re9 renamed RE9
- net rf0 renamed RF0
- net rf1 renamed RF1
- net rf12 renamed RF12
- net rf13 renamed RF13
- net rf2 renamed RF2
- net rf3 renamed RF3
- net rf4 renamed RF4
- net rf5 renamed RF5
- net rf8 renamed RF8
- net rg0 renamed RG0
- net rg1 renamed RG1
- net rg12 renamed RG12
- net rg13 renamed RG13
- net rg14 renamed RG14
- net rg15 renamed RG15
- net rg6 renamed RG6
- net rg7 renamed RG7
- net rg8 renamed RG8
- net rg9 renamed RG9
Changed lines of the file:
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@@
 		)
 	)
-	(hierarchical_label "rb10"
+	(hierarchical_label "RB10"
 		(shape input)
 		(at 189.865 67.31 0)
@@
 		)
 	)
-	(hierarchical_label "rg9"
+	(hierarchical_label "RG9"
 		(shape input)
 		(at 90.805 135.89 180)
@@
 		)
 	)
-	(hierarchical_label "rf8"
+	(hierarchical_label "RF8"
 		(shape input)
 		(at 189.865 143.51 0)
@@
 		)
 	)
-	(hierarchical_label "ra15"
+	(hierarchical_label "RA15"
 		(shape input)
 		(at 90.805 62.23 180)
@@
 		)
 	)
-	(hierarchical_label "re9"
+	(hierarchical_label "RE9"
 		(shape input)
 		(at 90.805 113.03 180)
@@
 		)
 	)
-	(hierarchical_label "rd11"
+	(hierarchical_label "RD11"
 		(shape input)
 		(at 189.865 113.03 0)
@@
 		)
 	)
-	(hierarchical_label "rg12"
+	(hierarchical_label "RG12"
 		(shape input)
 		(at 90.805 138.43 180)
@@
 		)
 	)
-	(hierarchical_label "re6"
+	(hierarchical_label "RE6"
 		(shape input)
 		(at 90.805 105.41 180)
@@
 		)
 	)
-	(hierarchical_label "rg1"
+	(hierarchical_label "RG1"
 		(shape input)
 		(at 90.805 120.65 180)
@@
 		)
 	)
-	(hierarchical_label "rd8"
+	(hierarchical_label "RD8"
 		(shape input)
 		(at 189.865 105.41 0)
@@
 		)
 	)
-	(hierarchical_label "rg15"
+	(hierarchical_label "RG15"
 		(shape input)
 		(at 90.805 146.05 180)
@@
 		)
 	)
-	(hierarchical_label "rg13"
+	(hierarchical_label "RG13"
 		(shape input)
 		(at 90.805 140.97 180)
@@
 		)
 	)
-	(hierarchical_label "rf1"
+	(hierarchical_label "RF1"
 		(shape input)
 		(at 189.865 130.81 0)
@@
 		)
 	)
-	(hierarchical_label "rc14"
+	(hierarchical_label "RC14"
 		(shape input)
 		(at 90.805 82.55 180)
@@
 		)
 	)
-	(hierarchical_label "rc13"
+	(hierarchical_label "RC13"
 		(shape input)
 		(at 90.805 80.01 180)
@@
 		)
 	)
-	(hierarchical_label "ra6"
+	(hierarchical_label "RA6"
 		(shape input)
 		(at 90.805 49.53 180)
@@
 		)
 	)
-	(hierarchical_label "re7"
+	(hierarchical_label "RE7"
 		(shape input)
 		(at 90.805 107.95 180)
@@
 		)
 	)
-	(hierarchical_label "rd15"
+	(hierarchical_label "RD15"
 		(shape input)
 		(at 189.865 123.19 0)
@@
 		)
 	)
-	(hierarchical_label "rb9"
+	(hierarchical_label "RB9"
 		(shape input)
 		(at 189.865 64.77 0)
@@
 		)
 	)
-	(hierarchical_label "ra9"
+	(hierarchical_label "RA9"
 		(shape input)
 		(at 90.805 54.61 180)
@@
 		)
 	)
-	(hierarchical_label "rd14"
+	(hierarchical_label "RD14"
 		(shape input)
 		(at 189.865 120.65 0)
@@
 		)
 	)
-	(hierarchical_label "ra7"
+	(hierarchical_label "RA7"
 		(shape input)
 		(at 90.805 52.07 180)
@@
 		)
 	)
-	(hierarchical_label "mclr"
+	(hierarchical_label "MCLR"
 		(shape input)
 		(at 189.865 36.83 0)
@@
 		)
 	)
-	(hierarchical_label "rb13"
+	(hierarchical_label "RB13"
 		(shape input)
 		(at 189.865 74.93 0)
@@
 		)
 	)
-	(hierarchical_label "rg8"
+	(hierarchical_label "RG8"
 		(shape input)
 		(at 90.805 133.35 180)
@@
 		)
 	)
-	(hierarchical_label "rd9"
+	(hierarchical_label "RD9"
 		(shape input)
 		(at 189.865 107.95 0)
@@
 		)
 	)
-	(hierarchical_label "re8"
+	(hierarchical_label "RE8"
 		(shape input)
 		(at 90.805 110.49 180)
@@
 		)
 	)
-	(hierarchical_label "rf4"
+	(hierarchical_label "RF4"
 		(shape input)
 		(at 189.865 138.43 0)
@@
 		)
 	)
-	(hierarchical_label "osc1"
+	(hierarchical_label "OSC1"
 		(shape input)
 		(at 80.645 77.47 180)
@@
 		)
 	)
-	(hierarchical_label "osc2"
+	(hierarchical_label "OSC2"
 		(shape input)
 		(at 80.645 85.09 180)
@@
 		)
 	)
-	(hierarchical_label "rf2"
+	(hierarchical_label "RF2"
 		(shape input)
 		(at 189.865 133.35 0)
@@
 		)
 	)
-	(hierarchical_label "vbus"
+	(hierarchical_label "VBUS"
 		(shape input)
 		(at 80.772 151.003 180)
@@
 		)
 	)
-	(hierarchical_label "rd10"
+	(hierarchical_label "RD10"
 		(shape input)
 		(at 189.865 110.49 0)
@@
 		)
 	)
-	(hierarchical_label "rg0"
+	(hierarchical_label "RG0"
 		(shape input)
 		(at 90.805 118.11 180)
@@
 		)
 	)
-	(hierarchical_label "rf13"
+	(hierarchical_label "RF13"
 		(shape input)
 		(at 189.865 148.59 0)
@@
 		)
 	)
-	(hierarchical_label "rd13"
+	(hierarchical_label "RD13"
 		(shape input)
 		(at 189.865 118.11 0)
@@
 		)
 	)
-	(hierarchical_label "rg14"
+	(hierarchical_label "RG14"
 		(shape input)
 		(at 90.805 143.51 180)
@@
 		)
 	)
-	(hierarchical_label "rf12"
+	(hierarchical_label "RF12"
 		(shape input)
 		(at 189.865 146.05 0)
@@
 		)
 	)
-	(hierarchical_label "rf5"
+	(hierarchical_label "RF5"
 		(shape input)
 		(at 189.865 140.97 0)
@@
 		)
 	)
-	(hierarchical_label "rg7"
+	(hierarchical_label "RG7"
 		(shape input)
 		(at 90.805 130.81 180)
@@
 		)
 	)
-	(hierarchical_label "ra10"
+	(hierarchical_label "RA10"
 		(shape input)
 		(at 90.805 57.15 180)
@@
 		)
 	)
-	(hierarchical_label "rb14"
+	(hierarchical_label "RB14"
 		(shape input)
 		(at 189.865 77.47 0)
@@
 		)
 	)
-	(hierarchical_label "rb11"
+	(hierarchical_label "RB11"
 		(shape input)
 		(at 189.865 69.85 0)
@@
 		)
 	)
-	(hierarchical_label "rf0"
+	(hierarchical_label "RF0"
 		(shape input)
 		(at 189.865 128.27 0)
@@
 		)
 	)
-	(hierarchical_label "rg6"
+	(hierarchical_label "RG6"
 		(shape input)
 		(at 90.805 128.27 180)
@@
 		)
 	)
-	(hierarchical_label "rd12"
+	(hierarchical_label "RD12"
 		(shape input)
 		(at 189.865 115.57 0)
@@
 		)
 	)
-	(hierarchical_label "rb12"
+	(hierarchical_label "RB12"
 		(shape input)
 		(at 189.865 72.39 0)
@@
 		)
 	)
-	(hierarchical_label "ra14"
+	(hierarchical_label "RA14"
 		(shape input)
 		(at 90.805 59.69 180)
@@
 		)
 	)
-	(hierarchical_label "rb8"
+	(hierarchical_label "RB8"
 		(shape input)
 		(at 189.865 62.23 0)
@@
 		)
 	)
-	(hierarchical_label "rb15"
+	(hierarchical_label "RB15"
 		(shape input)
 		(at 189.865 80.01 0)
@@
 		)
 	)
-	(hierarchical_label "rf3"
+	(hierarchical_label "RF3"
 		(shape input)
 		(at 189.865 135.89 0)
