File: amper_volt_meter.kicad_pcb (KiCad board)
At the start: 2 copper layers, 99.6 x 99.6 mm, 119 parts, among them J1 Conn_02x15_Odd_Even, J1001 buttons, J1002 buttons, J1003 buttons, J1004 buttons, J1005 buttons, J204 USB_B_Mini, J205 pickit, J301 OledSpiST1306, J302 OledSpiST7789, J501 potenciometer_digital_0, J502 potenciometer_digital_0, J503 potenciometer_digital_0, J504 potenciometer_digital_0, J701 OledSpiST7789, J702 OledSpiST1306, J801 tp?, J802 tp?, J803 tp?, J804 tp?, J805 tp?, J806 tp?, Q1 Q_NPN_BCE, SW1001 switch, SW1002 switch, SW1003 switch, SW1004 switch, SW1005 switch, U1 74HC595, U1101 ., U201 PIC18F46J50-I_PT, U501 MCP41010, U502 MCP41010, U503 MCP41010, U505 MCP41010, U601 LM1117DT-3.3, U801 LM358, Y201 Crystal_GND24_Small

Commit message: feat: migrar a KiCad 10 y reemplazar 0603 por 0805 - actualizar versiones de archivos y footprints SMD
Parts:
- C1101, C1102, C1103, C1104, C1105, C1106, C1107, C1108, C1109, C201, C202, C203, C204, C601, C602, C603, C604, C605, C606, C607: footprint Capacitor_SMD:C_0603_1608Metric -> Capacitor_SMD:C_0805_2012Metric
- R1001, R1002, R1003, R1004, R1005, R1006, R1007, R1008, R1009, R1010, R202, R203, R301, R302, R701, R702, R901, R902, R903, R904: footprint Resistor_SMD:R_0603_1608Metric -> Resistor_SMD:R_0805_2012Metric
