File: ucontroller_pic18F46j50.kicad_sch (KiCad schematic)
At the start: 11 parts, among them J204 USB_B_Mini, U201 PIC18F46J50-I_PT

Commit message: feat: migrar a KiCad 10 y reemplazar 0603 por 0805 - actualizar versiones de archivos y footprints SMD
Parts:
- C? (x4): footprint Capacitor_SMD:C_0603_1608Metric -> Capacitor_SMD:C_0805_2012Metric
- R? (x2): footprint Resistor_SMD:R_0603_1608Metric -> Resistor_SMD:R_0805_2012Metric
- gave numbers to parts that had none: 2
