File: ucontroller_pic18F46j50.kicad_sch (KiCad schematic)
At the start: 11 parts, among them J204 USB_B_Mini, J205 pickit, U201 PIC18F46J50-I_PT, Y201 Crystal_GND24_Small

Commit message: feat: agregar hierarchical_labels con nombres correctos a oS_AnaloDev (DiscoveryAnalog3) - 30 pines
Parts:
- gave numbers to parts that had none: 7
Changed lines of the file:
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@@
 		(dnp no)
 		(fields_autoplaced yes)
-		(property "Reference" "#PWR?"
+		(property "Reference" "#PWR0207"
 			(at 202.819 145.034 0)
 			(hide yes)
@@
 				(path "/606ef755-236d-4283-a129-fc8150c20746/b0ca9638-e9a2-4d8a-9c73-ce5c437e0625"
 					(reference "#PWR0207")
-					(unit 1)
-				)
-				(path "/606ef755-236d-4283-a129-fc8150c20746/c7d419ee-db35-4680-9f83-e183810d9dc3"
-					(reference "#PWR?")
 					(unit 1)
 				)
@@
 		(dnp no)
 		(fields_autoplaced yes)
-		(property "Reference" "#PWR?"
+		(property "Reference" "#PWR0202"
 			(at 52.705 70.485 0)
 			(hide yes)
@@
 				(path "/606ef755-236d-4283-a129-fc8150c20746/b0ca9638-e9a2-4d8a-9c73-ce5c437e0625"
 					(reference "#PWR0202")
-					(unit 1)
-				)
-				(path "/606ef755-236d-4283-a129-fc8150c20746/c7d419ee-db35-4680-9f83-e183810d9dc3"
-					(reference "#PWR?")
 					(unit 1)
 				)
@@
 		(dnp no)
 		(fields_autoplaced yes)
-		(property "Reference" "#PWR?"
+		(property "Reference" "#PWR0201"
 			(at 47.752 115.189 0)
 			(hide yes)
@@
 				(path "/606ef755-236d-4283-a129-fc8150c20746/b0ca9638-e9a2-4d8a-9c73-ce5c437e0625"
 					(reference "#PWR0201")
-					(unit 1)
-				)
-				(path "/606ef755-236d-4283-a129-fc8150c20746/c7d419ee-db35-4680-9f83-e183810d9dc3"
-					(reference "#PWR?")
 					(unit 1)
 				)
@@
 		(dnp no)
 		(fields_autoplaced yes)
-		(property "Reference" "C?"
+		(property "Reference" "C202"
 			(at 72.644 76.962 0)
 			(show_name no)
@@
 				(path "/606ef755-236d-4283-a129-fc8150c20746/b0ca9638-e9a2-4d8a-9c73-ce5c437e0625"
 					(reference "C202")
-					(unit 1)
-				)
-				(path "/606ef755-236d-4283-a129-fc8150c20746/c7d419ee-db35-4680-9f83-e183810d9dc3"
-					(reference "C?")
 					(unit 1)
 				)
@@
 		(dnp no)
 		(fields_autoplaced yes)
-		(property "Reference" "J?"
+		(property "Reference" "J205"
 			(at 245.4402 44.0944 0)
 			(show_name no)
@@
 				(path "/606ef755-236d-4283-a129-fc8150c20746/b0ca9638-e9a2-4d8a-9c73-ce5c437e0625"
 					(reference "J205")
-					(unit 1)
-				)
-				(path "/606ef755-236d-4283-a129-fc8150c20746/c7d419ee-db35-4680-9f83-e183810d9dc3"
-					(reference "J?")
 					(unit 1)
 				)
@@
 		(dnp no)
 		(fields_autoplaced yes)
-		(property "Reference" "#PWR?"
+		(property "Reference" "#PWR0204"
 			(at 68.961 156.972 0)
 			(hide yes)
@@
 				(path "/606ef755-236d-4283-a129-fc8150c20746/b0ca9638-e9a2-4d8a-9c73-ce5c437e0625"
 					(reference "#PWR0204")
-					(unit 1)
-				)
-				(path "/606ef755-236d-4283-a129-fc8150c20746/c7d419ee-db35-4680-9f83-e183810d9dc3"
-					(reference "#PWR?")
 					(unit 1)
 				)
@@
 		(in_pos_files yes)
 		(dnp no)
-		(property "Reference" "R?"
+		(property "Reference" "R201"
 			(at 251.46 79.375 90)
 			(show_name no)
@@
 				(path "/606ef755-236d-4283-a129-fc8150c20746/b0ca9638-e9a2-4d8a-9c73-ce5c437e0625"
 					(reference "R201")
-					(unit 1)
-				)
-				(path "/606ef755-236d-4283-a129-fc8150c20746/c7d419ee-db35-4680-9f83-e183810d9dc3"
-					(reference "R?")
 					(unit 1)
 				)
@@
 		(in_pos_files yes)
 		(dnp no)
-		(property "Reference" "C?"
+		(property "Reference" "C201"
 			(at 42.672 95.123 0)
 			(show_name no)
@@
 				(path "/606ef755-236d-4283-a129-fc8150c20746/b0ca9638-e9a2-4d8a-9c73-ce5c437e0625"
 					(reference "C201")
-					(unit 1)
-				)
-				(path "/606ef755-236d-4283-a129-fc8150c20746/c7d419ee-db35-4680-9f83-e183810d9dc3"
-					(reference "C?")
 					(unit 1)
 				)
@@
 		(dnp no)
 		(fields_autoplaced yes)
-		(property "Reference" "#PWR?"
+		(property "Reference" "#PWR0211"
 			(at 272.669 63.119 0)
 			(hide yes)
@@
 				(path "/606ef755-236d-4283-a129-fc8150c20746/b0ca9638-e9a2-4d8a-9c73-ce5c437e0625"
 					(reference "#PWR0211")
-					(unit 1)
-				)
-				(path "/606ef755-236d-4283-a129-fc8150c20746/c7d419ee-db35-4680-9f83-e183810d9dc3"
-					(reference "#PWR?")
 					(unit 1)
 				)
@@
 		(dnp no)
 		(fields_autoplaced yes)
-		(property "Reference" "C?"
+		(property "Reference" "C204"
 			(at 85.471 137.922 0)
 			(show_name no)
@@
 				(path "/606ef755-236d-4283-a129-fc8150c20746/b0ca9638-e9a2-4d8a-9c73-ce5c437e0625"
 					(reference "C204")
-					(unit 1)
-				)
-				(path "/606ef755-236d-4283-a129-fc8150c20746/c7d419ee-db35-4680-9f83-e183810d9dc3"
-					(reference "C?")
 					(unit 1)
 				)
@@
 		(dnp no)
 		(fields_autoplaced yes)
-		(property "Reference" "Y?"
+		(property "Reference" "Y201"
 			(at 74.295 68.8341 0)
 			(show_name no)
@@
 				(path "/606ef755-236d-4283-a129-fc8150c20746/b0ca9638-e9a2-4d8a-9c73-ce5c437e0625"
 					(reference "Y201")
-					(unit 1)
-				)
-				(path "/606ef755-236d-4283-a129-fc8150c20746/c7d419ee-db35-4680-9f83-e183810d9dc3"
-					(reference "Y?")
 					(unit 1)
 				)
@@
 		(dnp no)
 		(fields_autoplaced yes)
-		(property "Reference" "#PWR?"
+		(property "Reference" "#PWR0209"
 			(at 257.937 83.693 0)
 			(hide yes)
@@
 		(instances
 			(project "amper_volt_meter"
-				(path "/606ef755-236d-4283-a129-fc8150c20746/283e249b-17fa-4123-ad59-a4970e9d33a5"
-					(reference "#PWR?")
-					(unit 1)
-				)
 				(path "/606ef755-236d-4283-a129-fc8150c20746/b0ca9638-e9a2-4d8a-9c73-ce5c437e0625"
 					(reference "#PWR0209")
-					(unit 1)
-				)
-				(path "/606ef755-236d-4283-a129-fc8150c20746/f62fc848-fb80-4104-826c-eb02129eaaef"
-					(reference "#PWR?")
 					(unit 1)
 				)
@@
 		(dnp no)
 		(fields_autoplaced yes)
-		(property "Reference" "#PWR?"
+		(property "Reference" "#PWR0206"
 			(at 200.279 35.179 0)
 			(hide yes)
@@
 				(path "/606ef755-236d-4283-a129-fc8150c20746/b0ca9638-e9a2-4d8a-9c73-ce5c437e0625"
 					(reference "#PWR0206")
-					(unit 1)
-				)
-				(path "/606ef755-236d-4283-a129-fc8150c20746/c7d419ee-db35-4680-9f83-e183810d9dc3"
-					(reference "#PWR?")
 					(unit 1)
 				)
@@
 		(dnp no)
 		(fields_autoplaced yes)
-		(property "Reference" "#PWR?"
+		(property "Reference" "#PWR0210"
 			(at 266.319 45.339 0)
 			(hide yes)
@@
 				(path "/606ef755-236d-4283-a129-fc8150c20746/b0ca9638-e9a2-4d8a-9c73-ce5c437e0625"
 					(reference "#PWR0210")
-					(unit 1)
-				)
-				(path "/606ef755-236d-4283-a129-fc8150c20746/c7d419ee-db35-4680-9f83-e183810d9dc3"
-					(reference "#PWR?")
 					(unit 1)
 				)
@@
 		(dnp no)
 		(fields_autoplaced yes)
-		(property "Reference" "#PWR?"
+		(property "Reference" "#PWR0208"
 			(at 240.03 112.522 0)
 			(hide yes)
@@
 				(path "/606ef755-236d-4283-a129-fc8150c20746/b0ca9638-e9a2-4d8a-9c73-ce5c437e0625"
 					(reference "#PWR0208")
-					(unit 1)
-				)
-				(path "/606ef755-236d-4283-a129-fc8150c20746/c7d419ee-db35-4680-9f83-e183810d9dc3"
-					(reference "#PWR?")
 					(unit 1)
 				)
@@
 		(in_pos_files yes)
 		(dnp no)
-		(property "Reference" "R?"
+		(property "Reference" "R202"
 			(at 251.333 95.504 90)
 			(show_name no)
@@
 				(path "/606ef755-236d-4283-a129-fc8150c20746/b0ca9638-e9a2-4d8a-9c73-ce5c437e0625"
 					(reference "R202")
-					(unit 1)
-				)
-				(path "/606ef755-236d-4283-a129-fc8150c20746/c7d419ee-db35-4680-9f83-e183810d9dc3"
-					(reference "R?")
 					(unit 1)
 				)
@@
 		(dnp no)
 		(fields_autoplaced yes)
-		(property "Reference" "#PWR?"
+		(property "Reference" "#PWR0205"
 			(at 81.661 156.972 0)
 			(hide yes)
@@
 				(path "/606ef755-236d-4283-a129-fc8150c20746/b0ca9638-e9a2-4d8a-9c73-ce5c437e0625"
 					(reference "#PWR0205")
-					(unit 1)
-				)
-				(path "/606ef755-236d-4283-a129-fc8150c20746/c7d419ee-db35-4680-9f83-e183810d9dc3"
-					(reference "#PWR?")
 					(unit 1)
 				)
@@
 		(dnp no)
 		(fields_autoplaced yes)
-		(property "Reference" "#PWR?"
+		(property "Reference" "#PWR0203"
 			(at 59.436 90.043 0)
 			(hide yes)
@@
 				(path "/606ef755-236d-4283-a129-fc8150c20746/b0ca9638-e9a2-4d8a-9c73-ce5c437e0625"
 					(reference "#PWR0203")
-					(unit 1)
-				)
-				(path "/606ef755-236d-4283-a129-fc8150c20746/c7d419ee-db35-4680-9f83-e183810d9dc3"
-					(reference "#PWR?")
 					(unit 1)
 				)
@@
 		(dnp no)
 		(fields_autoplaced yes)
-		(property "Reference" "C?"
+		(property "Reference" "C203"
 			(at 72.771 137.922 0)
 			(show_name no)
@@
 				(path "/606ef755-236d-4283-a129-fc8150c20746/b0ca9638-e9a2-4d8a-9c73-ce5c437e0625"
 					(reference "C203")
-					(unit 1)
-				)
-				(path "/606ef755-236d-4283-a129-fc8150c20746/c7d419ee-db35-4680-9f83-e183810d9dc3"
-					(reference "C?")
 					(unit 1)
 				)
@@
 		(in_pos_files yes)
 		(dnp no)
-		(property "Reference" "R?"
+		(property "Reference" "R203"
 			(at 255.27 84.455 90)
 			(show_name no)
@@
 					(unit 1)
 				)
-				(path "/606ef755-236d-4283-a129-fc8150c20746/c7d419ee-db35-4680-9f83-e183810d9dc3"
-					(reference "R?")
-					(unit 1)
-				)

Commit message: feat: agregar 31 pines jerarquicos al sheet pic18F46j50 - ordenados por puerto (15 izq + 16 der)
Parts:
- C204: value 100n -> 1U
Connections:
- net mclr renamed MCLR
- net pgc renamed PGC
- net pgd renamed PGD
Changed lines of the file:
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@@
 		)
 	)
-	(hierarchical_label "pgd"
+	(hierarchical_label "PGD"
 		(shape input)
 		(at 194.818 70.358 0)
@@
 		)
 		(property "Intersheetrefs" "${INTERSHEET_REFS}"
-			(at 201.1708 70.358 0)
+			(at 194.818 71.628 0)
 			(hide yes)
 			(show_name no)
@@
 		)
 	)
-	(hierarchical_label "pgc"
+	(hierarchical_label "PGC"
 		(shape input)
 		(at 262.2296 59.3344 0)
@@
 		)
 		(property "Intersheetrefs" "${INTERSHEET_REFS}"
-			(at 268.522 59.3344 0)
+			(at 262.2296 60.6044 0)
 			(hide yes)
 			(show_name no)
@@
 		)
 	)
-	(hierarchical_label "mclr"
+	(hierarchical_label "MCLR"
 		(shape input)
 		(at 88.138 47.498 180)
@@
 		)
 		(property "Intersheetrefs" "${INTERSHEET_REFS}"
-			(at 80.9989 47.498 0)
+			(at 88.138 48.768 0)
 			(hide yes)
 			(show_name no)
@@
 		)
 	)
-	(hierarchical_label "mclr"
+	(hierarchical_label "MCLR"
 		(shape input)
 		(at 256.6416 49.1744 0)
@@
 		)
 		(property "Intersheetrefs" "${INTERSHEET_REFS}"
-			(at 263.7807 49.1744 0)
+			(at 256.6416 50.4444 0)
 			(hide yes)
 			(show_name no)
@@
 		)
 	)
-	(hierarchical_label "pgd"
+	(hierarchical_label "PGD"
 		(shape input)
 		(at 262.1534 56.7944 0)
@@
 		)
 		(property "Intersheetrefs" "${INTERSHEET_REFS}"
-			(at 268.5062 56.7944 0)
+			(at 262.1534 58.0644 0)
 			(hide yes)
 			(show_name no)
@@
 		)
 	)
-	(hierarchical_label "pgc"
+	(hierarchical_label "PGC"
 		(shape input)
 		(at 194.818 67.818 0)
@@
 		)
 		(property "Intersheetrefs" "${INTERSHEET_REFS}"
-			(at 201.1104 67.818 0)
+			(at 194.818 69.088 0)
 			(hide yes)
 			(show_name no)
@@
 		(fields_autoplaced yes)
 		(property "Reference" "C204"
-			(at 85.471 137.922 0)
+			(at 85.09 137.9219 0)
 			(show_name no)
 			(do_not_autoplace no)
@@
 			)
 		)
-		(property "Value" "100n"
-			(at 85.471 140.462 0)
-			(show_name no)
-			(do_not_autoplace no)
+		(property "Value" "1U"
+			(at 85.09 140.4619 0)
+			(show_name no)
+			(do_not_autoplace no)
