File: Digital_Control.kicad_sch (KiCad schematic)
At the start: 20 parts, among them J501 potenciometer_digital_0, J502 potenciometer_digital_0, J503 potenciometer_digital_0, J504 potenciometer_digital_0, U501 MCP41010, U502 MCP41010, U503 MCP41010, U505 MCP41010

Commit message: feat: agregar hierarchical_labels con nombres correctos a oS_AnaloDev (DiscoveryAnalog3) - 30 pines
Parts:
- gave numbers to parts that had none: 12
Changed lines of the file:
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@@
 		(dnp no)
 		(fields_autoplaced yes)
-		(property "Reference" "#PWR?"
+		(property "Reference" "#PWR0501"
 			(at 55.753 131.953 0)
 			(hide yes)
@@
 				(path "/606ef755-236d-4283-a129-fc8150c20746/0b301535-cd84-4a21-805d-be4f537ebfda"
 					(reference "#PWR0501")
-					(unit 1)
-				)
-				(path "/606ef755-236d-4283-a129-fc8150c20746/74c3696e-dda9-4e41-9c02-5e756dc00ace"
-					(reference "#PWR?")
 					(unit 1)
 				)
@@
 		(in_pos_files yes)
 		(dnp no)
-		(property "Reference" "R?"
+		(property "Reference" "R511"
 			(at 226.822 96.012 90)
 			(show_name no)
@@
 				(path "/606ef755-236d-4283-a129-fc8150c20746/0b301535-cd84-4a21-805d-be4f537ebfda"
 					(reference "R511")
-					(unit 1)
-				)
-				(path "/606ef755-236d-4283-a129-fc8150c20746/74c3696e-dda9-4e41-9c02-5e756dc00ace"
-					(reference "R?")
 					(unit 1)
 				)
@@
 		(in_pos_files yes)
 		(dnp no)
-		(property "Reference" "R?"
+		(property "Reference" "R512"
 			(at 227.203 101.6 90)
 			(show_name no)
@@
 					(unit 1)
 				)
-				(path "/606ef755-236d-4283-a129-fc8150c20746/74c3696e-dda9-4e41-9c02-5e756dc00ace"
-					(reference "R?")
-					(unit 1)
-				)
 			)
 			(project "rpi2w_epaper_zigbee"
@@
 		(in_pos_files yes)
 		(dnp no)
-		(property "Reference" "R?"
+		(property "Reference" "R510"
 			(at 176.022 108.458 90)
 			(show_name no)
@@
 					(unit 1)
 				)
-				(path "/606ef755-236d-4283-a129-fc8150c20746/74c3696e-dda9-4e41-9c02-5e756dc00ace"
-					(reference "R?")
-					(unit 1)
-				)
 			)
 			(project "rpi2w_epaper_zigbee"
@@
 		(in_pos_files yes)
 		(dnp no)
-		(property "Reference" "R?"
+		(property "Reference" "R508"
 			(at 175.641 96.393 90)
 			(show_name no)
@@
 					(unit 1)
 				)
-				(path "/606ef755-236d-4283-a129-fc8150c20746/74c3696e-dda9-4e41-9c02-5e756dc00ace"
-					(reference "R?")
-					(unit 1)
-				)
 			)
 			(project "rpi2w_epaper_zigbee"
@@
 		(in_pos_files yes)
 		(dnp no)
-		(property "Reference" "R?"
+		(property "Reference" "R503"
 			(at 84.074 101.473 90)
 			(show_name no)
@@
 				(path "/606ef755-236d-4283-a129-fc8150c20746/0b301535-cd84-4a21-805d-be4f537ebfda"
 					(reference "R503")
-					(unit 1)
-				)
-				(path "/606ef755-236d-4283-a129-fc8150c20746/74c3696e-dda9-4e41-9c02-5e756dc00ace"
-					(reference "R?")
 					(unit 1)
 				)
@@
 		(dnp no)
 		(fields_autoplaced yes)
-		(property "Reference" "#PWR?"
+		(property "Reference" "#PWR0502"
 			(at 114.935 71.628 0)
 			(hide yes)
@@
 				(path "/606ef755-236d-4283-a129-fc8150c20746/0b301535-cd84-4a21-805d-be4f537ebfda"
 					(reference "#PWR0502")
-					(unit 1)
-				)
-				(path "/606ef755-236d-4283-a129-fc8150c20746/74c3696e-dda9-4e41-9c02-5e756dc00ace"
-					(reference "#PWR?")
 					(unit 1)
 				)
@@
 		(in_pos_files yes)
 		(dnp no)
-		(property "Reference" "R?"
+		(property "Reference" "R509"
 			(at 175.895 102.362 90)
 			(show_name no)
@@
 				(path "/606ef755-236d-4283-a129-fc8150c20746/0b301535-cd84-4a21-805d-be4f537ebfda"
 					(reference "R509")
-					(unit 1)
-				)
-				(path "/606ef755-236d-4283-a129-fc8150c20746/74c3696e-dda9-4e41-9c02-5e756dc00ace"
-					(reference "R?")
 					(unit 1)
 				)
@@
 		(in_pos_files yes)
 		(dnp no)
-		(property "Reference" "R?"
+		(property "Reference" "R507"
 			(at 130.302 107.569 90)
 			(show_name no)
@@
 				(path "/606ef755-236d-4283-a129-fc8150c20746/0b301535-cd84-4a21-805d-be4f537ebfda"
 					(reference "R507")
-					(unit 1)
-				)
-				(path "/606ef755-236d-4283-a129-fc8150c20746/74c3696e-dda9-4e41-9c02-5e756dc00ace"
-					(reference "R?")
 					(unit 1)
 				)
@@
 		(in_pos_files yes)
 		(dnp no)
-		(property "Reference" "R?"
+		(property "Reference" "R505"
 			(at 129.921 95.504 90)
 			(show_name no)
@@
 				(path "/606ef755-236d-4283-a129-fc8150c20746/0b301535-cd84-4a21-805d-be4f537ebfda"
 					(reference "R505")
-					(unit 1)
-				)
-				(path "/606ef755-236d-4283-a129-fc8150c20746/74c3696e-dda9-4e41-9c02-5e756dc00ace"
-					(reference "R?")
 					(unit 1)
 				)
@@
 		(in_pos_files yes)
 		(dnp no)
-		(property "Reference" "R?"
+		(property "Reference" "R513"
 			(at 227.33 107.696 90)
 			(show_name no)
@@
 					(unit 1)
 				)
-				(path "/606ef755-236d-4283-a129-fc8150c20746/74c3696e-dda9-4e41-9c02-5e756dc00ace"
-					(reference "R?")
-					(unit 1)
-				)
 			)
 			(project "rpi2w_epaper_zigbee"
@@
 		(in_pos_files yes)
 		(dnp no)
-		(property "Reference" "R?"
+		(property "Reference" "R502"
 			(at 83.693 96.393 90)
 			(show_name no)
@@
 					(unit 1)
 				)
-				(path "/606ef755-236d-4283-a129-fc8150c20746/74c3696e-dda9-4e41-9c02-5e756dc00ace"
-					(reference "R?")
-					(unit 1)
-				)
 			)
 			(project "rpi2w_epaper_zigbee"
@@
 		(in_pos_files yes)
 		(dnp no)
-		(property "Reference" "R?"
+		(property "Reference" "R506"
 			(at 130.175 101.473 90)
 			(show_name no)
@@
 					(unit 1)
 				)
-				(path "/606ef755-236d-4283-a129-fc8150c20746/74c3696e-dda9-4e41-9c02-5e756dc00ace"
-					(reference "R?")
-					(unit 1)
-				)
 			)
 			(project "rpi2w_epaper_zigbee"
@@
 		(in_pos_files yes)
 		(dnp no)
-		(property "Reference" "R?"
+		(property "Reference" "R504"
 			(at 84.074 108.204 90)
 			(show_name no)
@@
 					(unit 1)
 				)
-				(path "/606ef755-236d-4283-a129-fc8150c20746/74c3696e-dda9-4e41-9c02-5e756dc00ace"
-					(reference "R?")
-					(unit 1)
-				)
