File: Display_LCD.kicad_sch (KiCad schematic)
At the start: 9 parts, among them Q1 Q_NPN_BCE, U1 74HC595

Commit message: feat: agregar hierarchical_labels con nombres correctos a oS_AnaloDev (DiscoveryAnalog3) - 30 pines
Parts:
- gave numbers to parts that had none: 5
Changed lines of the file:
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@@
 		(dnp no)
 		(fields_autoplaced yes)
-		(property "Reference" "#PWR0901"
+		(property "Reference" "#PWR03"
 			(at 149.5552 139.2936 0)
 			(hide yes)
@@
 				(path "/606ef755-236d-4283-a129-fc8150c20746/2914e67b-33d9-4834-b079-0a9220979c82"
 					(reference "#PWR03")
-					(unit 1)
-				)
-				(path "/606ef755-236d-4283-a129-fc8150c20746/c7d419ee-db35-4680-9f83-e183810d9dc3"
-					(reference "#PWR0901")
 					(unit 1)
 				)
@@
 		(dnp no)
 		(fields_autoplaced yes)
-		(property "Reference" "#PWR0901"
+		(property "Reference" "#PWR08"
 			(at 174.3964 104.5464 0)
 			(hide yes)
@@
 				(path "/606ef755-236d-4283-a129-fc8150c20746/2914e67b-33d9-4834-b079-0a9220979c82"
 					(reference "#PWR08")
-					(unit 1)
-				)
-				(path "/606ef755-236d-4283-a129-fc8150c20746/c7d419ee-db35-4680-9f83-e183810d9dc3"
-					(reference "#PWR0901")
 					(unit 1)
 				)
@@
 		(in_pos_files yes)
 		(dnp no)
-		(property "Reference" "R?"
+		(property "Reference" "R4"
 			(at 87.1728 94.4372 90)
 			(show_name no)
@@
 			)
 			(project "amper_volt_meter"
-				(path "/606ef755-236d-4283-a129-fc8150c20746/283e249b-17fa-4123-ad59-a4970e9d33a5"
-					(reference "R701")
-					(unit 1)
-				)
 				(path "/606ef755-236d-4283-a129-fc8150c20746/2914e67b-33d9-4834-b079-0a9220979c82"
 					(reference "R4")
-					(unit 1)
-				)
-				(path "/606ef755-236d-4283-a129-fc8150c20746/f62fc848-fb80-4104-826c-eb02129eaaef"
-					(reference "R?")
 					(unit 1)
 				)
@@
 					(unit 1)
 				)
-				(path "/606ef755-236d-4283-a129-fc8150c20746/f62fc848-fb80-4104-826c-eb02129eaaef"
-					(reference "DS1")
-					(unit 1)
-				)
 			)
 		)
@@
 		(dnp no)
 		(fields_autoplaced yes)
-		(property "Reference" "#PWR0901"
+		(property "Reference" "#PWR09"
 			(at 93.5228 104.5972 0)
 			(hide yes)
@@
 				(path "/606ef755-236d-4283-a129-fc8150c20746/2914e67b-33d9-4834-b079-0a9220979c82"
 					(reference "#PWR09")
-					(unit 1)
-				)
-				(path "/606ef755-236d-4283-a129-fc8150c20746/c7d419ee-db35-4680-9f83-e183810d9dc3"
-					(reference "#PWR0901")
 					(unit 1)
 				)
@@
 		(dnp no)
 		(fields_autoplaced yes)
-		(property "Reference" "#PWR?"
+		(property "Reference" "#PWR07"
 			(at 216.7636 121.0056 0)
 			(hide yes)
@@
 		(instances
 			(project "amper_volt_meter"
-				(path "/606ef755-236d-4283-a129-fc8150c20746/283e249b-17fa-4123-ad59-a4970e9d33a5"
-					(reference "#PWR0702")
-					(unit 1)
-				)
 				(path "/606ef755-236d-4283-a129-fc8150c20746/2914e67b-33d9-4834-b079-0a9220979c82"
 					(reference "#PWR07")
-					(unit 1)
-				)
-				(path "/606ef755-236d-4283-a129-fc8150c20746/f62fc848-fb80-4104-826c-eb02129eaaef"
-					(reference "#PWR?")
 					(unit 1)
 				)
@@
 		(dnp no)
 		(fields_autoplaced yes)
-		(property "Reference" "#PWR?"
+		(property "Reference" "#PWR05"
 			(at 131.1148 91.3892 0)
 			(hide yes)
@@
 		(instances
 			(project "amper_volt_meter"
-				(path "/606ef755-236d-4283-a129-fc8150c20746/283e249b-17fa-4123-ad59-a4970e9d33a5"
-					(reference "#PWR0702")
-					(unit 1)
-				)
 				(path "/606ef755-236d-4283-a129-fc8150c20746/2914e67b-33d9-4834-b079-0a9220979c82"
 					(reference "#PWR05")
-					(unit 1)
-				)
-				(path "/606ef755-236d-4283-a129-fc8150c20746/f62fc848-fb80-4104-826c-eb02129eaaef"
-					(reference "#PWR?")
 					(unit 1)
 				)
@@
 		(dnp no)
 		(fields_autoplaced yes)
-		(property "Reference" "#PWR0901"
+		(property "Reference" "#PWR04"
 			(at 193.802 141.6812 0)
 			(hide yes)
@@
 				(path "/606ef755-236d-4283-a129-fc8150c20746/2914e67b-33d9-4834-b079-0a9220979c82"
 					(reference "#PWR04")
-					(unit 1)
-				)
-				(path "/606ef755-236d-4283-a129-fc8150c20746/c7d419ee-db35-4680-9f83-e183810d9dc3"
-					(reference "#PWR0901")
 					(unit 1)
 				)
@@
 		(in_pos_files yes)
 		(dnp no)
-		(property "Reference" "R?"
+		(property "Reference" "R3"
 			(at 87.1728 79.1972 90)
 			(show_name no)
@@
 			)
 			(project "amper_volt_meter"
-				(path "/606ef755-236d-4283-a129-fc8150c20746/283e249b-17fa-4123-ad59-a4970e9d33a5"
-					(reference "R701")
-					(unit 1)
-				)
 				(path "/606ef755-236d-4283-a129-fc8150c20746/2914e67b-33d9-4834-b079-0a9220979c82"
 					(reference "R3")
-					(unit 1)
-				)
-				(path "/606ef755-236d-4283-a129-fc8150c20746/f62fc848-fb80-4104-826c-eb02129eaaef"
-					(reference "R?")
 					(unit 1)
 				)
@@
 		(dnp no)
 		(fields_autoplaced yes)
-		(property "Reference" "#PWR?"
+		(property "Reference" "#PWR010"
 			(at 93.5228 79.1972 0)
 			(hide yes)
@@
 		(instances
 			(project "amper_volt_meter"
-				(path "/606ef755-236d-4283-a129-fc8150c20746/283e249b-17fa-4123-ad59-a4970e9d33a5"
-					(reference "#PWR0702")
-					(unit 1)
-				)
 				(path "/606ef755-236d-4283-a129-fc8150c20746/2914e67b-33d9-4834-b079-0a9220979c82"
 					(reference "#PWR010")
-					(unit 1)
-				)
-				(path "/606ef755-236d-4283-a129-fc8150c20746/f62fc848-fb80-4104-826c-eb02129eaaef"
-					(reference "#PWR?")
 					(unit 1)
 				)
@@
 		(in_pos_files yes)
 		(dnp no)
-		(property "Reference" "R?"
+		(property "Reference" "R1"
 			(at 124.7648 93.5228 90)
 			(show_name no)
@@
 			)
 			(project "amper_volt_meter"
-				(path "/606ef755-236d-4283-a129-fc8150c20746/283e249b-17fa-4123-ad59-a4970e9d33a5"
-					(reference "R701")
-					(unit 1)
-				)
 				(path "/606ef755-236d-4283-a129-fc8150c20746/2914e67b-33d9-4834-b079-0a9220979c82"
 					(reference "R1")
-					(unit 1)
-				)
-				(path "/606ef755-236d-4283-a129-fc8150c20746/f62fc848-fb80-4104-826c-eb02129eaaef"
-					(reference "R?")
 					(unit 1)
 				)
@@
 		(in_pos_files yes)
 		(dnp no)
-		(property "Reference" "R?"
+		(property "Reference" "R5"
 			(at 102.9716 93.1672 90)
 			(show_name no)
@@
 			)
 			(project "amper_volt_meter"
-				(path "/606ef755-236d-4283-a129-fc8150c20746/283e249b-17fa-4123-ad59-a4970e9d33a5"
-					(reference "R701")
-					(unit 1)
-				)
 				(path "/606ef755-236d-4283-a129-fc8150c20746/2914e67b-33d9-4834-b079-0a9220979c82"
 					(reference "R5")
-					(unit 1)
-				)
-				(path "/606ef755-236d-4283-a129-fc8150c20746/f62fc848-fb80-4104-826c-eb02129eaaef"
-					(reference "R?")
 					(unit 1)
 				)
@@
 		(dnp no)
 		(fields_autoplaced yes)
-		(property "Reference" "#PWR?"
+		(property "Reference" "#PWR01"
 			(at 149.5552 90.7796 0)
 			(hide yes)
@@
 		(instances
 			(project "amper_volt_meter"
-				(path "/606ef755-236d-4283-a129-fc8150c20746/283e249b-17fa-4123-ad59-a4970e9d33a5"
-					(reference "#PWR0702")
-					(unit 1)
-				)
 				(path "/606ef755-236d-4283-a129-fc8150c20746/2914e67b-33d9-4834-b079-0a9220979c82"
 					(reference "#PWR01")
-					(unit 1)
-				)
-				(path "/606ef755-236d-4283-a129-fc8150c20746/f62fc848-fb80-4104-826c-eb02129eaaef"
-					(reference "#PWR?")
 					(unit 1)
 				)
@@
 		(in_pos_files yes)
 		(dnp no)
-		(property "Reference" "R?"
+		(property "Reference" "R2"
 			(at 118.618 116.0272 90)
 			(show_name no)
@@
 			)
 			(project "amper_volt_meter"
-				(path "/606ef755-236d-4283-a129-fc8150c20746/283e249b-17fa-4123-ad59-a4970e9d33a5"
-					(reference "R701")
-					(unit 1)
-				)
 				(path "/606ef755-236d-4283-a129-fc8150c20746/2914e67b-33d9-4834-b079-0a9220979c82"
 					(reference "R2")
-					(unit 1)
-				)
-				(path "/606ef755-236d-4283-a129-fc8150c20746/f62fc848-fb80-4104-826c-eb02129eaaef"
-					(reference "R?")
 					(unit 1)
 				)
@@
 		(dnp no)
 		(fields_autoplaced yes)
-		(property "Reference" "#PWR0901"
+		(property "Reference" "#PWR06"
 			(at 132.6388 122.3772 0)
 			(hide yes)
@@
 				(path "/606ef755-236d-4283-a129-fc8150c20746/2914e67b-33d9-4834-b079-0a9220979c82"
 					(reference "#PWR06")
-					(unit 1)
-				)
-				(path "/606ef755-236d-4283-a129-fc8150c20746/c7d419ee-db35-4680-9f83-e183810d9dc3"
-					(reference "#PWR0901")
 					(unit 1)
 				)
@@
 		(dnp no)
 		(fields_autoplaced yes)
-		(property "Reference" "#PWR?"
+		(property "Reference" "#PWR02"
 			(at 193.802 102.0064 0)
 			(hide yes)
@@
 		(instances
 			(project "amper_volt_meter"
-				(path "/606ef755-236d-4283-a129-fc8150c20746/283e249b-17fa-4123-ad59-a4970e9d33a5"
-					(reference "#PWR0702")
-					(unit 1)
-				)
 				(path "/606ef755-236d-4283-a129-fc8150c20746/2914e67b-33d9-4834-b079-0a9220979c82"
 					(reference "#PWR02")
 					(unit 1)
 				)
-				(path "/606ef755-236d-4283-a129-fc8150c20746/f62fc848-fb80-4104-826c-eb02129eaaef"
-					(reference "#PWR?")
-					(unit 1)
-				)
