File: Power_Distribution.kicad_sch (KiCad schematic)
At the start: 9 parts

Commit message: feat: migrar a KiCad 10 y reemplazar 0603 por 0805 - actualizar versiones de archivos y footprints SMD
Parts:
- C? (x7): footprint Capacitor_SMD:C_0603_1608Metric -> Capacitor_SMD:C_0805_2012Metric
- gave numbers to parts that had none: 2

Commit message: feat: agregar hierarchical_labels con nombres correctos a oS_AnaloDev (DiscoveryAnalog3) - 30 pines
Parts:
- gave numbers to parts that had none: 7
Changed lines of the file:
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@@
 		(dnp no)
 		(fields_autoplaced yes)
-		(property "Reference" "#PWR?"
+		(property "Reference" "#PWR0605"
 			(at 163.322 75.438 0)
 			(hide yes)
@@
 					(unit 1)
 				)
-				(path "/606ef755-236d-4283-a129-fc8150c20746/c7d419ee-db35-4680-9f83-e183810d9dc3"
-					(reference "#PWR?")
-					(unit 1)
-				)
 			)
 			(project "rpi2w_epaper_zigbee"
@@
 		(dnp no)
 		(fields_autoplaced yes)
-		(property "Reference" "JP?"
+		(property "Reference" "JP601"
 			(at 98.933 92.71 0)
 			(show_name no)
@@
 					(unit 1)
 				)
-				(path "/606ef755-236d-4283-a129-fc8150c20746/c7d419ee-db35-4680-9f83-e183810d9dc3"
-					(reference "JP?")
-					(unit 1)
-				)
 			)
 			(project "rpi2w_epaper_zigbee"
@@
 		(dnp no)
 		(fields_autoplaced yes)
-		(property "Reference" "C?"
+		(property "Reference" "C607"
 			(at 202.819 101.727 0)
 			(show_name no)
@@
 					(unit 1)
 				)
-				(path "/606ef755-236d-4283-a129-fc8150c20746/c7d419ee-db35-4680-9f83-e183810d9dc3"
-					(reference "C?")
-					(unit 1)
-				)
 			)
 			(project "rpi2w_epaper_zigbee"
@@
 		(dnp no)
 		(fields_autoplaced yes)
-		(property "Reference" "U?"
+		(property "Reference" "U601"
 			(at 111.633 100.33 0)
 			(show_name no)
@@
 					(unit 1)
 				)
-				(path "/606ef755-236d-4283-a129-fc8150c20746/c7d419ee-db35-4680-9f83-e183810d9dc3"
-					(reference "U?")
-					(unit 1)
-				)
 			)
 			(project "rpi2w_epaper_zigbee"
@@
 		(dnp no)
 		(fields_autoplaced yes)
-		(property "Reference" "C?"
+		(property "Reference" "C603"
 			(at 155.702 56.388 0)
 			(show_name no)
@@
 					(unit 1)
 				)
-				(path "/606ef755-236d-4283-a129-fc8150c20746/c7d419ee-db35-4680-9f83-e183810d9dc3"
-					(reference "C?")
-					(unit 1)
-				)
 			)
 			(project "rpi2w_epaper_zigbee"
@@
 		(dnp no)
 		(fields_autoplaced yes)
-		(property "Reference" "C?"
+		(property "Reference" "C601"
 			(at 97.663 109.22 0)
 			(show_name no)
@@
 					(unit 1)
 				)
-				(path "/606ef755-236d-4283-a129-fc8150c20746/c7d419ee-db35-4680-9f83-e183810d9dc3"
-					(reference "C?")
-					(unit 1)
-				)
 			)
 			(project "rpi2w_epaper_zigbee"
@@
 		(dnp no)
 		(fields_autoplaced yes)
-		(property "Reference" "C?"
+		(property "Reference" "C604"
 			(at 167.132 56.388 0)
 			(show_name no)
@@
 					(unit 1)
 				)
-				(path "/606ef755-236d-4283-a129-fc8150c20746/c7d419ee-db35-4680-9f83-e183810d9dc3"
-					(reference "C?")
-					(unit 1)
-				)
 			)
 			(project "rpi2w_epaper_zigbee"
@@
 		(dnp no)
 		(fields_autoplaced yes)
-		(property "Reference" "#PWR?"
+		(property "Reference" "#PWR0607"
 			(at 199.009 123.317 0)
 			(hide yes)
@@
 					(unit 1)
 				)
-				(path "/606ef755-236d-4283-a129-fc8150c20746/c7d419ee-db35-4680-9f83-e183810d9dc3"
-					(reference "#PWR?")
-					(unit 1)
-				)
 			)
 			(project "rpi2w_epaper_zigbee"
@@
 		(dnp no)
 		(fields_autoplaced yes)
-		(property "Reference" "#PWR?"
+		(property "Reference" "#PWR0606"
 			(at 186.309 123.317 0)
 			(hide yes)
@@
 					(unit 1)
 				)
-				(path "/606ef755-236d-4283-a129-fc8150c20746/c7d419ee-db35-4680-9f83-e183810d9dc3"
-					(reference "#PWR?")
-					(unit 1)
-				)
 			)
 			(project "rpi2w_epaper_zigbee"
@@
 		(dnp no)
 		(fields_autoplaced yes)
-		(property "Reference" "#PWR?"
+		(property "Reference" "#PWR0604"
 			(at 151.892 51.308 0)
 			(hide yes)
@@
 					(unit 1)
 				)
-				(path "/606ef755-236d-4283-a129-fc8150c20746/c7d419ee-db35-4680-9f83-e183810d9dc3"
-					(reference "#PWR?")
-					(unit 1)
-				)
 			)
 			(project "rpi2w_epaper_zigbee"
@@
 		(dnp no)
 		(fields_autoplaced yes)
-		(property "Reference" "C?"
+		(property "Reference" "C605"
 			(at 179.832 56.388 0)
 			(show_name no)
@@
 					(unit 1)
 				)
-				(path "/606ef755-236d-4283-a129-fc8150c20746/c7d419ee-db35-4680-9f83-e183810d9dc3"
-					(reference "C?")
-					(unit 1)
-				)
 			)
 			(project "rpi2w_epaper_zigbee"
@@
 		(dnp no)
 		(fields_autoplaced yes)
-		(property "Reference" "#PWR?"
+		(property "Reference" "#PWR0608"
 			(at 210.439 86.487 0)
 			(hide yes)
@@
 					(unit 1)
 				)
-				(path "/606ef755-236d-4283-a129-fc8150c20746/c7d419ee-db35-4680-9f83-e183810d9dc3"
-					(reference "#PWR?")
-					(unit 1)
-				)
 			)
 			(project "rpi2w_epaper_zigbee"
@@
 		(dnp no)
 		(fields_autoplaced yes)
-		(property "Reference" "#PWR?"
+		(property "Reference" "#PWR0603"
 			(at 128.143 101.6 0)
 			(hide yes)
@@
 					(unit 1)
 				)
-				(path "/606ef755-236d-4283-a129-fc8150c20746/c7d419ee-db35-4680-9f83-e183810d9dc3"
-					(reference "#PWR?")
-					(unit 1)
-				)
 			)
 			(project "rpi2w_epaper_zigbee"
@@
 		(dnp no)
 		(fields_autoplaced yes)
-		(property "Reference" "C?"
+		(property "Reference" "C602"
 			(at 131.953 110.49 0)
 			(show_name no)
@@
 					(unit 1)
 				)
-				(path "/606ef755-236d-4283-a129-fc8150c20746/c7d419ee-db35-4680-9f83-e183810d9dc3"
-					(reference "C?")
-					(unit 1)
-				)
 			)
 			(project "rpi2w_epaper_zigbee"
@@
 		(dnp no)
 		(fields_autoplaced yes)
-		(property "Reference" "#PWR?"
+		(property "Reference" "#PWR0602"
 			(at 111.633 125.73 0)
 			(hide yes)
@@
 					(unit 1)
 				)
-				(path "/606ef755-236d-4283-a129-fc8150c20746/c7d419ee-db35-4680-9f83-e183810d9dc3"
-					(reference "#PWR?")
-					(unit 1)
-				)
 			)
 			(project "rpi2w_epaper_zigbee"
@@
 		(dnp no)
 		(fields_autoplaced yes)
-		(property "Reference" "#PWR?"
+		(property "Reference" "#PWR0601"
 			(at 82.423 120.65 0)
 			(hide yes)
@@
 					(unit 1)
 				)
-				(path "/606ef755-236d-4283-a129-fc8150c20746/c7d419ee-db35-4680-9f83-e183810d9dc3"
-					(reference "#PWR?")
-					(unit 1)
-				)
 			)
 			(project "rpi2w_epaper_zigbee"
@@
 		(dnp no)
 		(fields_autoplaced yes)
-		(property "Reference" "C?"
+		(property "Reference" "C606"
 			(at 190.119 101.727 0)
 			(show_name no)
@@
 					(unit 1)
 				)
-				(path "/606ef755-236d-4283-a129-fc8150c20746/c7d419ee-db35-4680-9f83-e183810d9dc3"
-					(reference "C?")
-					(unit 1)
-				)
