File: amper_volt_meter.kicad_sch (KiCad schematic)
At the start: 0 parts

Commit message: fix: PIM100 sheet - tamaño correcto 55x119mm, pines en bordes del rectangulo sin lineas zigzag
Other:
- sheet PIM100 ports: added none; removed AMPER, BLK_RPI, DC_RPI, GPIO20, GPIO21, GPIO22, GPIO23, GPIO24, RES_RPI, SCL_1, SCL_2, SDA_1, SDA_2
