File: amper_volt_meter.kicad_sch (KiCad schematic)
At the start: 0 parts

Commit message: feat: agregar 31 pines jerarquicos al sheet pic18F46j50 - ordenados por puerto (15 izq + 16 der)
Other:
- sheet ucontroller_pic18F46j50 renamed pic18F46j50
- sheet DiscoveryAnalog3 ports: added AI1+/OSC1 (1+), AI2+/OSC12(1+), AWG1 (W1), D1, D2, D3, D4, D5, D6, D7, D8, DC Output 1 (V1), DC Output 2 (V2), DO10 (10), DO9 (9), GND/AI1, GND/AI2, INT/CLK1 (C1), INT/CLK2 (C2), SDI/SDO (P1), SDI/SDO/UART_TX (P2), SPI_CLK/UART_CTS (P3), SPI_CS/UART_RTS/PWM1 (P4), Trigger Input (T1), Trigger Output (T0), UART_RX/PWM2 (P5); removed none
- sheet pic18F46j50 ports: added AN10, AN11, AN8, AN9, MCLR, PGC, PGD, RA0, RA1, RA5, RB0, RC0, RC1, RC6, RC7, RD2, RD3, RD4, RD5, RD6, RD7, RE0, RE1, RE2, SCL_1, SCL_2, SDA_1, SDA_2, VDD_CORE, VREF+, VREF-; removed none

Commit message: fix: pines jerarquicos fuera del rectangulo (offset 2.54mm) + documentar defecto zig-zag en LEARNINGS.md
Other:
- sheet pic18F46j50 renamed ucontroller_pic18F46j50
